File: Hardware/V1/ESP32-S3-Remote/ESP32-S3-Remote.kicad_pcb (KiCad board)
At the start: 2 copper layers, 55 parts, among them J1 Conn_01x12_Pin, J2 Conn_01x04_Pin, J3 Conn_01x04_Pin, P1 USB_C_Plug_USB2.0, Q1 BSS138, Q10 BSS138, Q11 BSS138, Q12 BSS138, Q13 BSS138, Q2 BSS138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

Commit message: Make layout
Parts:
- removed P1: USB_C_Plug_USB2.0, Connector_USB:USB_C_Receptacle_GCT_USB4110
- added C7: 100n, Capacitor_SMD:C_0603_1608Metric, F.Cu at (101.1, 95.9)
- added J4: USB_C_Receptacle_USB2.0_14P, Connector_USB:USB_C_Receptacle_GCT_USB4110, F.Cu at (93.5, 104.1)
- added R27: 5.1k, Resistor_SMD:R_0603_1608Metric, F.Cu at (87.3, 96.0)
- added R28: 5.1k, Resistor_SMD:R_0603_1608Metric, F.Cu at (92.3, 96.0)
- moved Q6 64.6 mm to (106.9, 91.5)
- moved Q7 63.6 mm to (106.9, 95.1)
- moved Q8 62.7 mm to (106.9, 98.6)
- moved Q11 62.3 mm to (72.6, 95.5), turned to 180 degrees
- moved J2 61.7 mm to (65.8, 99.7), turned to 180 degrees
- moved Q9 61.7 mm to (106.9, 102.1)
- moved J3 57.1 mm to (65.8, 91.6), turned to 180 degrees
- moved Q12 54.3 mm to (72.6, 91.9), turned to 180 degrees
- moved Q1 52.5 mm to (106.9, 73.8)
- moved Q2 51.7 mm to (106.9, 77.4)
- moved U1 51.5 mm to (91.4, 74.6)
- moved Q3 50.9 mm to (106.9, 80.9)
- moved Q4 50.1 mm to (106.9, 84.5)
- moved Q5 49.3 mm to (106.9, 88.0)
- moved J1 49.2 mm to (116.1, 79.1)
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Routing:
- net GND: track 0.00 -> 56.7 mm, vias 0 -> 49
- net +3.3V: track 0.00 -> 47.8 mm, vias 0 -> 2
- net /LEVEL_UP: track 0.00 -> 43.7 mm, vias 0 -> 9
- net /ESP_BOOT: track 0.00 -> 39.1 mm, vias 0 -> 2
- net /LEVEL_75_TRIG: track 0.00 -> 36.7 mm, vias 0 -> 2
- net /LEVEL_50_TRIG: track 0.00 -> 34.1 mm, vias 0 -> 2
- net /LEVEL_25_TRIG: track 0.00 -> 31.0 mm, vias 0 -> 2
- net /ALL_TRIG: track 0.00 -> 28.8 mm, vias 0 -> 2
- net /LEVEL_0_TRIG: track 0.00 -> 27.9 mm, vias 0 -> 2
- net /CH3_TRIG: track 0.00 -> 27.6 mm, vias 0 -> 2
- net /CH2_TRIG: track 0.00 -> 27.4 mm, vias 0 -> 2
- net /CH1_TRIG: track 0.00 -> 26.7 mm, vias 0 -> 2
- net /LEVEL_100_TRIG: track 0.00 -> 26.2 mm, vias 0 -> 2
- net Net-(U2-EN): track 0.00 -> 26.0 mm, vias 0 -> 2
- net /UP_TRIG: track 0.00 -> 24.9 mm, vias 0 -> 2
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- added copper zone on B.Cu, net GND
- added copper zone on F.Cu, net GND
Other:
- board outline added: 54 x 40 mm
- board text added: "Dylan Collaud"
- board text added: "Remote V2 06.2026"

Commit message: Order files
Parts:
- added TP1: TestPoint, TestPoint:TestPoint_Pad_D1.5mm, F.Cu at (67.1, 75.9)
- added TP2: TestPoint, TestPoint:TestPoint_Pad_D1.5mm, F.Cu at (71.1, 103.1)
Routing:
- net GND: vias 49 -> 59
